File: mainboard_v3.kicad_sch (KiCad schematic)
At the start: 37 parts, among them J1 PWR_IN, J3 PLD, J4 PLD, J5 IO, J6 IO, J7 DEBUG, SW1 RESET, U1 W65C02SxP, U2 CY62256-70PC, U3 28C256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

Commit message: Update
Parts:
- C7, C8: value (none) -> 0.1uF; footprint (none) -> Capacitor_THT:C_Disc_D3.0mm_W1.6mm_P2.50mm
Other:
- note added: "FIX: Replace D3 with wire to have ~{RST} on expansion port FIX: U4 already includes pull-up. Remove RN2C from board"
- note added: "FIX: Replace useless fuse with wire"

Commit message: Update
Parts:
- C1: footprint (none) -> Capacitor_THT:CP_Radial_D6.3mm_P2.50mm
- U1: symbol 65xx:W65C02SxP -> mainboard_v3:W65C02SxP
- U4: symbol AK's_Library:DS1813 -> mainboard_v3:DS1813
- U7: symbol 65xx:W65C22SxP -> mainboard_v3:W65C22SxP
Changed lines of the file:
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@@
     (effects (font (size 1.27 1.27)) (justify right bottom))
   )
-  (symbol (lib_id "65xx:W65C02SxP") (at 62.23 118.11 0) (unit 1)
+  (symbol (lib_id "mainboard_v3:W65C02SxP") (at 62.23 118.11 0) (unit 1)
     (in_bom yes) (on_board yes)
     (property "Reference" "U1" (id 0) (at 62.23 101.6 0))
@@
     (pin "9")
   )
-  (symbol (lib_id "AK's_Library:DS1813") (at 29.21 57.15 0) (unit 1)
+  (symbol (lib_id "mainboard_v3:DS1813") (at 29.21 57.15 0) (unit 1)
     (in_bom yes) (on_board yes)
     (property "Reference" "U4" (id 0) (at 23.368 55.9816 0)
@@
     (pin "1")
   )
-  (symbol (lib_id "65xx:W65C22SxP") (at 203.2 118.11 0) (unit 1)
+  (symbol (lib_id "mainboard_v3:W65C22SxP") (at 203.2 118.11 0) (unit 1)
     (in_bom yes) (on_board yes)
     (property "Reference" "U7" (id 0) (at 194.31 85.09 0))
@@
       (effects (font (size 1.27 1.27)) (justify left))
     )
-    (property "Footprint" "" (id 2) (at 67.0052 184.15 0)
+    (property "Footprint" "Capacitor_THT:CP_Radial_D6.3mm_P2.50mm" (id 2) (at 67.0052 184.15 0)
       (effects (font (size 1.27 1.27)) hide)
     )
@@
   (symbol (lib_id "power:GND") (at 261.62 24.13 0) (unit 1)
     (in_bom yes) (on_board yes)
-    (property "Reference" "#PWR?" (id 0) (at 261.62 30.48 0)
+    (property "Reference" "#PWR0102" (id 0) (at 261.62 30.48 0)
       (effects (font (size 1.27 1.27)) hide)
     )
@@
   (symbol (lib_id "power:VCC") (at 236.22 31.75 0) (unit 1)
     (in_bom yes) (on_board yes)
-    (property "Reference" "#PWR?" (id 0) (at 236.22 35.56 0)
+    (property "Reference" "#PWR0106" (id 0) (at 236.22 35.56 0)
       (effects (font (size 1.27 1.27)) hide)
     )
@@
   (symbol (lib_id "power:GND") (at 236.22 36.83 0) (unit 1)
     (in_bom yes) (on_board yes)
-    (property "Reference" "#PWR?" (id 0) (at 236.22 43.18 0)
+    (property "Reference" "#PWR0105" (id 0) (at 236.22 43.18 0)
       (effects (font (size 1.27 1.27)) hide)
     )
@@
   (symbol (lib_id "power:VCC") (at 261.62 19.05 0) (unit 1)
     (in_bom yes) (on_board yes)
-    (property "Reference" "#PWR?" (id 0) (at 261.62 22.86 0)
+    (property "Reference" "#PWR0104" (id 0) (at 261.62 22.86 0)
       (effects (font (size 1.27 1.27)) hide)
     )
@@
   (symbol (lib_id "power:VCC") (at 186.69 101.6 0) (unit 1)
     (in_bom yes) (on_board yes)
-    (property "Reference" "#PWR?" (id 0) (at 186.69 105.41 0)
+    (property "Reference" "#PWR0101" (id 0) (at 186.69 105.41 0)
       (effects (font (size 1.27 1.27)) hide)
     )
@@
       (reference "#PWR030") (unit 1) (value "VCC") (footprint "")
     )
+    (path "/ced1d47f-2435-463b-9691-8bf82addfb1c"
+      (reference "#PWR0101") (unit 1) (value "VCC") (footprint "")
+    )
+    (path "/3b774e26-56b9-47d4-be90-1bb33439081b"
+      (reference "#PWR0102") (unit 1) (value "GND") (footprint "")
+    )
     (path "/00000000-0000-0000-0000-00006291d05c"
       (reference "#PWR0103") (unit 1) (value "GND") (footprint "")
     )
-    (path "/3b774e26-56b9-47d4-be90-1bb33439081b"
-      (reference "#PWR?") (unit 1) (value "GND") (footprint "")
+    (path "/861d0f8d-6c01-456c-b42c-587faf924a8b"
+      (reference "#PWR0104") (unit 1) (value "VCC") (footprint "")
+    )
+    (path "/5cba0742-1707-4a65-9f23-82d295b4f20c"
+      (reference "#PWR0105") (unit 1) (value "GND") (footprint "")
     )
     (path "/441e2f03-2bcb-42ed-a327-7c3e7d39e2e9"
-      (reference "#PWR?") (unit 1) (value "VCC") (footprint "")
-    )
-    (path "/5cba0742-1707-4a65-9f23-82d295b4f20c"
-      (reference "#PWR?") (unit 1) (value "GND") (footprint "")
-    )
-    (path "/861d0f8d-6c01-456c-b42c-587faf924a8b"
-      (reference "#PWR?") (unit 1) (value "VCC") (footprint "")
-    )
-    (path "/ced1d47f-2435-463b-9691-8bf82addfb1c"
-      (reference "#PWR?") (unit 1) (value "VCC") (footprint "")
+      (reference "#PWR0106") (unit 1) (value "VCC") (footprint "")
     )
     (path "/32ea78f4-956b-43c5-99f1-7d3c1958be2b"
-      (reference "C1") (unit 1) (value "10uF") (footprint "")
+      (reference "C1") (unit 1) (value "10uF") (footprint "Capacitor_THT:CP_Radial_D6.3mm_P2.50mm")
     )
     (path "/00000000-0000-0000-0000-000060e9182d"
